Commit message: Update Hexapod.urdf

File: Hexapod.urdf (robot description, URDF)
Before this commit: robot hex_3dof3, 19 links, 18 joints
Links:
- link Pata1_Link1: geometry collision mesh filename=meshes/Pata1_Link1.obj; visual mesh filename=meshes/Pata1_Link1.obj
- link Pata1_Link2: geometry collision mesh filename=meshes/Pata1_Link2.obj; visual mesh filename=meshes/Pata1_Link2.obj
- link Pata1_Link3: geometry collision mesh filename=meshes/Pata1_Link3.obj; collision sphere radius=0.0
- link Pata2_Link1: geometry collision mesh filename=meshes/Pata2_Link1.obj; visual mesh filename=meshes/Pata2_Link1.obj
- link Pata2_Link2: geometry collision mesh filename=meshes/Pata2_Link2.obj; visual mesh filename=meshes/Pata2_Link2.obj
- link Pata2_Link3: geometry collision mesh filename=meshes/Pata2_Link3.obj; collision sphere radius=0.0
- link Pata3_Link1: geometry collision mesh filename=meshes/Pata3_Link1.obj; visual mesh filename=meshes/Pata3_Link1.obj
- link Pata3_Link2: geometry collision mesh filename=meshes/Pata3_Link2.obj; visual mesh filename=meshes/Pata3_Link2.obj
- link Pata3_Link3: geometry collision mesh filename=meshes/Pata3_Link3.obj; collision sphere radius=0.0
- link Pata4_Link1: geometry collision mesh filename=meshes/Pata4_Link1.obj; visual mesh filename=meshes/Pata4_Link1.obj
- link Pata4_Link2: geometry collision mesh filename=meshes/Pata4_Link2.obj; visual mesh filename=meshes/Pata4_Link2.obj
- link Pata4_Link3: geometry collision mesh filename=meshes/Pata4_Link3.obj; collision sphere radius=0.0
- link Pata5_Link1: geometry collision mesh filename=meshes/Pata5_Link1.obj; visual mesh filename=meshes/Pata5_Link1.obj
- link Pata5_Link2: geometry collision mesh filename=meshes/Pata5_Link2.obj; visual mesh filename=meshes/Pata5_Link2.obj
- link Pata5_Link3: geometry collision mesh filename=meshes/Pata5_Link3.obj; visual mesh filename=meshes/Pata5_Link3.obj
- link Pata6_Link1: geometry collision mesh filename=meshes/Pata6_Link1.obj; visual mesh filename=meshes/Pata6_Link1.obj
- link Pata6_Link2: geometry collision mesh filename=meshes/Pata6_Link2.obj; visual mesh filename=meshes/Pata6_Link2.obj
- link Pata6_Link3: geometry collision mesh filename=meshes/Pata6_Link3.obj; collision sphere radius=0.0
- link base_link: geometry collision mesh filename=meshes/base_link.obj; visual mesh filename=meshes/base_link.obj
Joints:
- joint Pata1_Motor1: limit lower=-0.52 upper=0.52 effort=0 velocity=0.19 -> lower=-1.58 upper=1.58 effort=360 velocity=12
- joint Pata1_Motor2: limit lower=-0.52 upper=0.52 effort=0 velocity=0.19 -> lower=-1.58 upper=0.79 effort=360 velocity=12
- joint Pata1_Motor3: limit lower=-0.52 upper=0.52 effort=0 velocity=0.19 -> lower=-0.79 upper=1.58 effort=360 velocity=12
- joint Pata2_Motor1: limit lower=-0.52 upper=0.52 effort=0 velocity=0.19 -> lower=-1.58 upper=1.58 effort=360 velocity=12
- joint Pata2_Motor2: limit lower=-0.52 upper=0.52 effort=0 velocity=0.19 -> lower=-1.58 upper=0.79 effort=360 velocity=12
- joint Pata2_Motor3: limit lower=-0.52 upper=0.52 effort=0 velocity=0.19 -> lower=-0.79 upper=1.58 effort=360 velocity=12
- joint Pata3_Motor1: limit lower=-0.52 upper=0.52 effort=0 velocity=0.19 -> lower=-1.58 upper=1.58 effort=360 velocity=12
- joint Pata3_Motor2: limit lower=-0.52 upper=0.52 effort=0 velocity=0.19 -> lower=-1.58 upper=0.79 effort=360 velocity=12
- joint Pata3_Motor3: limit lower=-0.52 upper=0.52 effort=0 velocity=0.19 -> lower=-0.79 upper=1.58 effort=360 velocity=12; origin xyz=-0.058928 0 0 rpy=-3.1416 1.583E-15 0 -> xyz=-0.058928 0 0 rpy=3.1416 3.1416 0
- joint Pata4_Motor1: limit lower=-0.52 upper=0.52 effort=0 velocity=0.19 -> lower=-1.58 upper=1.58 effort=360 velocity=12
- joint Pata4_Motor2: limit lower=-0.52 upper=0.52 effort=0 velocity=0.19 -> lower=-1.58 upper=0.79 effort=360 velocity=12
- joint Pata4_Motor3: limit lower=-0.52 upper=0.52 effort=0 velocity=0.19 -> lower=-0.79 upper=1.58 effort=360 velocity=12
- joint Pata5_Motor1: limit lower=-0.52 upper=0.52 effort=0 velocity=0.19 -> lower=-1.58 upper=1.58 effort=360 velocity=12
- joint Pata5_Motor2: limit lower=-0.52 upper=0.52 effort=0 velocity=0.19 -> lower=-1.58 upper=0.79 effort=360 velocity=12
- joint Pata5_Motor3: limit lower=-0.52 upper=0.52 effort=0 velocity=0.19 -> lower=-0.79 upper=1.58 effort=360 velocity=12
- joint Pata6_Motor1: limit lower=-0.52 upper=0.52 effort=0 velocity=0.19 -> lower=-1.58 upper=1.58 effort=360 velocity=12
- joint Pata6_Motor2: limit lower=-0.52 upper=0.52 effort=0 velocity=0.19 -> lower=-1.58 upper=0.79 effort=360 velocity=12
- joint Pata6_Motor3: limit lower=-0.52 upper=0.52 effort=0 velocity=0.19 -> lower=-0.79 upper=1.58 effort=360 velocity=12
